File: tapestry-controller.kicad_pcb (KiCad board)
At the start: 2 copper layers, 160 x 120 mm, 21 parts, among them J1 LED_STRIP_8, J11 12-24V Barrel Jack, J12 +5V, J2 LED_STRIP_1, J3 LED_STRIP_2, J4 LED_STRIP_3, J5 LED_STRIP_4, J6 LED_STRIP_5, J7 LED_STRIP_6, J8 LED_STRIP_7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

Commit message: Updated to fix the upside down LCD
Parts:
- U5: footprint libs:SPI_Screen_320_x_240_dual -> libs:SPI_Screen_320_x_240_2.8
- moved U5 25.5 mm to (108.8, 70.1)
Routing:
- net +3V3: track 102.5 -> 62.7 mm
- net /RESET: track 112.7 -> 88.6 mm, vias 1 -> 0
- net /IO5: track 101.7 -> 89.4 mm
- net /IO18: track 105.1 -> 95.7 mm
- net /IO23: track 111.2 -> 102.9 mm
- net /DC: track 96.0 -> 89.5 mm, vias 1 -> 0
- net /CS_Disp: track 100.1 -> 98.8 mm, vias 1 -> 0
- net GND: vias 54 -> 39
