File: tapestry-controller.kicad_pcb (KiCad board)
At the start: 2 copper layers, 160 x 120 mm, 21 parts, among them J1 LED_STRIP_8, J11 12-24V Barrel Jack, J12 +5V, J2 LED_STRIP_1, J3 LED_STRIP_2, J4 LED_STRIP_3, J5 LED_STRIP_4, J6 LED_STRIP_5, J7 LED_STRIP_6, J8 LED_STRIP_7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

Commit message: Final Release Version
Parts:
- removed J9: LED_STRIP_9, libs:p2035a-dinkle-3-way-5mm
- added SW1: Reset, Button_Switch_SMD:SW_Push_1P1T_NO_6x6mm_H9.5mm, F.Cu at (92.2, 127.0)
- added SW2: Program, Button_Switch_SMD:SW_Push_1P1T_NO_6x6mm_H9.5mm, F.Cu at (160.0, 127.0)
- moved J1 6.28 mm to (181.0, 141.6)
- moved J2 6.28 mm to (76.0, 141.6)
- moved J3 6.28 mm to (91.0, 141.6)
- moved J4 6.28 mm to (106.0, 141.6)
- moved J5 6.28 mm to (121.0, 141.6)
- moved J6 6.28 mm to (136.0, 141.6)
- moved J7 6.28 mm to (151.0, 141.6)
- moved J8 6.28 mm to (166.0, 141.6)
Connections:
- U5 pad 8: /IO5 -> Net-(U5-Pad8)
Routing:
- net /IO21: track 141.4 -> 108.3 mm
- net /RESET: track 88.6 -> 105.0 mm
- net /IO22: track 124.3 -> 135.7 mm
- net /IO26: track 118.7 -> 125.0 mm
- net /IO15: track 85.9 -> 92.1 mm
- net /IO27: track 102.3 -> 108.6 mm
- net /IO14: track 69.4 -> 75.7 mm
- net /IO25: track 135.1 -> 141.4 mm
- net /IO4: track 54.3 -> 59.3 mm
- net +5V: track 60.0 -> 64.8 mm
- net /IO19: track 115.3 -> 120.0 mm
Other:
- net class Default removed
