File: tapestry-controller.sch (KiCad schematic (older format))
At the start: 19 parts, among them J1 LED_STRIP_8, J11 12-24V Barrel Jack, J12 +5V, J2 LED_STRIP_1, J3 LED_STRIP_2, J4 LED_STRIP_3, J5 LED_STRIP_4, J6 LED_STRIP_5, J7 LED_STRIP_6, J8 LED_STRIP_7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

Commit message: Updated to fix the upside down LCD
Parts:
- U5: footprint libs:SPI_Screen_320_x_240_dual -> libs:SPI_Screen_320_x_240_2.8
Changed lines of the file:
@@
 F 0 "U5" H 9400 2000 50  0000 R CNN
 F 1 "2.8tft" H 9500 1350 50  0000 R CNN
-F 2 "libs:SPI_Screen_320_x_240_dual" H 9650 1350 50  0001 C CNN
+F 2 "libs:SPI_Screen_320_x_240_2.8" H 9650 1350 50  0001 C CNN
 F 3 "" H 9650 1350 50  0001 C CNN
 	1    9650 1650

Commit message: Final Release Version
Parts:
- removed J9: LED_STRIP_9, libs:p2035a-dinkle-3-way-5mm, symbol Connector_Generic:Conn_01x03
- added SW1: Reset, Button_Switch_SMD:SW_Push_1P1T_NO_6x6mm_H9.5mm, symbol Switch:SW_Push
- added SW2: Program, Button_Switch_SMD:SW_Push_1P1T_NO_6x6mm_H9.5mm, symbol Switch:SW_Push
Connections:
- net GND: now also SW1.1, SW2.1
- net IO21: now also SW2.2
- net IO5: no longer U5.8 (LED)
- net RESET: now also SW1.2
- no-connect marks 11 -> 12
Changed lines of the file:
@@
 Text Label 10400 1600 2    50   ~ 0
 SCLK
-Text Label 10400 1700 2    50   ~ 0
+Text Label 10400 1800 2    50   ~ 0
 LED
 NoConn ~ 10050 1800
@@
 Wire Wire Line
 	7050 1200 7050 1300
-$Comp
-L Connector_Generic:Conn_01x03 J9
-U 1 1 61741C0E
-P 6550 2000
-F 0 "J9" H 6468 2317 50  0000 C CNN
-F 1 "LED_STRIP_9" H 6468 2226 50  0000 C CNN
-F 2 "libs:p2035a-dinkle-3-way-5mm" H 6550 2000 50  0001 C CNN
-F 3 "~" H 6550 2000 50  0001 C CNN
-	1    6550 2000
-	-1   0    0    -1
-$EndComp
-$Comp
-L power:GND #PWR0129
-U 1 1 61741FB0
-P 7050 2200
-F 0 "#PWR0129" H 7050 1950 50  0001 C CNN
-F 1 "GND" H 7055 2027 50  0000 C CNN
-F 2 "" H 7050 2200 50  0001 C CNN
-F 3 "" H 7050 2200 50  0001 C CNN
-	1    7050 2200
-	1    0    0    -1
-$EndComp
-$Comp
-L power:+5V #PWR0130
-U 1 1 61741FBA
-P 7050 1850
-F 0 "#PWR0130" H 7050 1700 50  0001 C CNN
-F 1 "+5V" H 7065 2023 50  0000 C CNN
-F 2 "" H 7050 1850 50  0001 C CNN
-F 3 "" H 7050 1850 50  0001 C CNN
-	1    7050 1850
-	1    0    0    -1
-$EndComp
-Wire Wire Line
-	6750 2000 6950 2000
-Wire Wire Line
-	6750 1900 7050 1900
-Wire Wire Line
-	7050 1900 7050 1850
-Wire Wire Line
-	6750 2100 7050 2100
-Wire Wire Line
-	7050 2100 7050 2200
 Wire Wire Line
 	3600 1150 3600 1200
@@
 Text Label 6950 1100 2    50   ~ 0
 IO22
-Text Label 6950 2000 2    50   ~ 0
-IO21
 Wire Wire Line
 	2850 1350 3450 1350
 Wire Wire Line
 	2850 1450 3450 1450
+Text Label 10400 1900 2    50   ~ 0
+SCLK
+NoConn ~ 10400 1700
+Text Label 10400 2000 2    50   ~ 0
+IO21
+Text Label 10400 2100 2    50   ~ 0
+MOSI
+Text Label 10400 2200 2    50   ~ 0
+LED
+Text Label 10400 2300 2    50   ~ 0
+IO22
+$Comp
+L Switch:SW_Push SW1
+U 1 1 618A85C3
+P 1800 3500
+F 0 "SW1" H 1800 3785 50  0000 C CNN
+F 1 "Reset" H 1800 3694 50  0000 C CNN
+F 2 "Button_Switch_SMD:SW_Push_1P1T_NO_6x6mm_H9.5mm" H 1800 3700 50  0001 C CNN
+F 3 "~" H 1800 3700 50  0001 C CNN
+	1    1800 3500
+	1    0    0    -1
+$EndComp
+$Comp
+L power:GND #PWR0133
+U 1 1 618A950E
+P 1500 3600
+F 0 "#PWR0133" H 1500 3350 50  0001 C CNN
+F 1 "GND" H 1505 3427 50  0000 C CNN
+F 2 "" H 1500 3600 50  0001 C CNN
+F 3 "" H 1500 3600 50  0001 C CNN
+	1    1500 3600
+	1    0    0    -1
+$EndComp
+Text Label 2300 3500 2    50   ~ 0
+RESET
+Wire Wire Line
+	1500 3600 1500 3500
+Wire Wire Line
+	1500 3500 1600 3500
+Wire Wire Line
+	2000 3500 2300 3500
+$Comp
+L Switch:SW_Push SW2
+U 1 1 618B5BBE
+P 2900 3500
+F 0 "SW2" H 2900 3785 50  0000 C CNN
+F 1 "Program" H 2900 3694 50  0000 C CNN
+F 2 "Button_Switch_SMD:SW_Push_1P1T_NO_6x6mm_H9.5mm" H 2900 3700 50  0001 C CNN
+F 3 "~" H 2900 3700 50  0001 C CNN
+	1    2900 3500
+	1    0    0    -1
+$EndComp
+$Comp
+L power:GND #PWR0129
+U 1 1 618B5F7A
+P 2600 3600
+F 0 "#PWR0129" H 2600 3350 50  0001 C CNN
+F 1 "GND" H 2605 3427 50  0000 C CNN
+F 2 "" H 2600 3600 50  0001 C CNN
+F 3 "" H 2600 3600 50  0001 C CNN
+	1    2600 3600
+	1    0    0    -1
+$EndComp
+Wire Wire Line
+	2600 3600 2600 3500
+Wire Wire Line
+	2600 3500 2700 3500
+Wire Wire Line
+	3100 3500 3400 3500
+Text Label 3400 3500 2    50   ~ 0
+IO21
 $EndSCHEMATC
